File: audio_jack.kicad_sch (KiCad schematic)
At the start: 5 parts, among them J2 AudioJack3_SwitchTR, J3 Conn_01x03, J4 AudioJack3_SwitchTR, J5 Conn_01x03

Commit message: complete layout
Connections:
- net LEFT_IN: now also RV1.5; no longer RV1.2
- net LEFT_OUT: now also J5.1 (Pin_1)
- net RIGHT_IN: now also RV1.2; no longer RV1.5
- net RIGHT_OUT: no longer J5.1 (Pin_1)
- net at J2.R, J3.1 (Pin_1): now also RV1.3; no longer RV1.6
- net at J2.T, J3.3 (Pin_3): now also RV1.6; no longer RV1.3
- net GND renamed GND_OPA
