File: op_amplifier_left.kicad_sch (KiCad schematic)
At the start: 6 parts, among them U3 NE5532

Commit message: complete layout
Parts:
- removed U3: NE5532, Package_DIP:DIP-8_W7.62mm_Socket, symbol Amplifier_Operational:NE5532
- added U3: NE5532, Package_DIP:DIP-8_W7.62mm_Socket, symbol Amplifier_Operational:NE5532
- C14: renamed from C10; footprint (none) -> Capacitor_THT:C_Rect_L10.0mm_W5.0mm_P5.00mm_P7.50mm
Connections:
- net at R6.1: now also U3.6 (-)
- net at C14.2, R5.1: now also U3.5 (+)
- net at R8.1: now also U3.7
- net GND renamed GND_OPA
Changed lines of the file:
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@@
+	)
+	(symbol
+		(lib_id "Device:R")
+		(at 85.09 85.09 0)
+		(unit 1)
+		(exclude_from_sim no)
+		(in_bom yes)
+		(on_board yes)
+		(dnp no)
+		(fields_autoplaced yes)
+		(property "Reference" "R5"
+			(at 87.63 83.8199 0)
+			(effects
+				(font
+					(size 1.27 1.27)
+				)
+				(justify left)
+			)
+		)
+		(property "Value" "100K"
+			(at 87.63 86.3599 0)
+			(effects
+				(font
+					(size 1.27 1.27)
+				)
+				(justify left)
+			)
+		)
+		(property "Footprint" "Resistor_THT:R_Axial_DIN0309_L9.0mm_D3.2mm_P12.70mm_Horizontal"
+			(at 83.312 85.09 90)
+			(effects
+				(font
+					(size 1.27 1.27)
+				)
+				(hide yes)
+			)
+		)
+		(property "Datasheet" "~"
+			(at 85.09 85.09 0)
+			(effects
+				(font
+					(size 1.27 1.27)
+				)
+				(hide yes)
+			)
+		)
+		(property "Description" "Resistor"
+			(at 85.09 85.09 0)
+			(effects
+				(font
+					(size 1.27 1.27)
+				)
+				(hide yes)
+			)
+		)
+		(pin "1"
+		)
+		(pin "2"
+		)
+		(instances
+			(project "headphone_amplifier_v0"
+				(path "/3983550c-3b96-4d77-b5c7-1354f8e757f8/406fb7ac-178d-4932-ad58-7c7a39bfab55"
+					(reference "R5")
+					(unit 1)
+				)
+			)
+		)
 	)
 	(symbol
@@
 		(dnp no)
 		(fields_autoplaced yes)
-		(property "Reference" "#PWR09"
+		(property "Reference" "#PWR07"
 			(at 97.79 102.87 0)
 			(effects
@@
 			)
 		)
-		(property "Value" "GND"
+		(property "Value" "GND_OPA"
 			(at 97.79 101.6 0)
 			(effects
@@
 			(project "headphone_amplifier_v0"
 				(path "/3983550c-3b96-4d77-b5c7-1354f8e757f8/406fb7ac-178d-4932-ad58-7c7a39bfab55"
-					(reference "#PWR09")
+					(reference "#PWR07")
 					(unit 1)
 				)
@@
 	(symbol
 		(lib_id "Device:R")
-		(at 85.09 85.09 0)
-		(unit 1)
-		(exclude_from_sim no)
-		(in_bom yes)
-		(on_board yes)
-		(dnp no)
-		(fields_autoplaced yes)
-		(property "Reference" "R5"
-			(at 87.63 83.8199 0)
-			(effects
-				(font
-					(size 1.27 1.27)
-				)
-				(justify left)
-			)
-		)
-		(property "Value" "100K"
-			(at 87.63 86.3599 0)
-			(effects
-				(font
-					(size 1.27 1.27)
-				)
-				(justify left)
+		(at 124.46 74.93 90)
+		(unit 1)
+		(exclude_from_sim no)
+		(in_bom yes)
+		(on_board yes)
+		(dnp no)
+		(fields_autoplaced yes)
+		(property "Reference" "R8"
+			(at 124.46 68.58 90)
+			(effects
+				(font
+					(size 1.27 1.27)
+				)
+			)
+		)
+		(property "Value" "R"
+			(at 124.46 71.12 90)
+			(effects
+				(font
+					(size 1.27 1.27)
+				)
 			)
 		)
 		(property "Footprint" "Resistor_THT:R_Axial_DIN0309_L9.0mm_D3.2mm_P12.70mm_Horizontal"
-			(at 83.312 85.09 90)
+			(at 124.46 76.708 90)
 			(effects
 				(font
@@
 		)
 		(property "Datasheet" "~"
-			(at 85.09 85.09 0)
+			(at 124.46 74.93 0)
 			(effects
 				(font
@@
 		)
 		(property "Description" "Resistor"
-			(at 85.09 85.09 0)
+			(at 124.46 74.93 0)
 			(effects
 				(font
@@
 			(project "headphone_amplifier_v0"
 				(path "/3983550c-3b96-4d77-b5c7-1354f8e757f8/406fb7ac-178d-4932-ad58-7c7a39bfab55"
-					(reference "R5")
+					(reference "R8")
+					(unit 1)
+				)
+			)
+		)
+	)
+	(symbol
+		(lib_id "Device:C")
+		(at 73.66 72.39 90)
+		(unit 1)
+		(exclude_from_sim no)
+		(in_bom yes)
+		(on_board yes)
+		(dnp no)
+		(fields_autoplaced yes)
+		(property "Reference" "C14"
+			(at 73.66 64.77 90)
+			(effects
+				(font
+					(size 1.27 1.27)
+				)
+			)
+		)
+		(property "Value" "0.1u"
+			(at 73.66 67.31 90)
+			(effects
+				(font
+					(size 1.27 1.27)
+				)
+			)
+		)
+		(property "Footprint" "Capacitor_THT:C_Rect_L10.0mm_W5.0mm_P5.00mm_P7.50mm"
+			(at 77.47 71.4248 0)
+			(effects
+				(font
+					(size 1.27 1.27)
+				)
+				(hide yes)
+			)
+		)
+		(property "Datasheet" "~"
+			(at 73.66 72.39 0)
+			(effects
+				(font
+					(size 1.27 1.27)
+				)
+				(hide yes)
+			)
+		)
+		(property "Description" "Unpolarized capacitor"
+			(at 73.66 72.39 0)
+			(effects
+				(font
+					(size 1.27 1.27)
+				)
+				(hide yes)
+			)
+		)
+		(pin "2"
+		)
+		(pin "1"
+		)
+		(instances
+			(project "headphone_amplifier_v0"
+				(path "/3983550c-3b96-4d77-b5c7-1354f8e757f8/406fb7ac-178d-4932-ad58-7c7a39bfab55"
+					(reference "C14")
 					(unit 1)
 				)
@@
 		(dnp no)
 		(fields_autoplaced yes)
-		(property "Reference" "#PWR08"
+		(property "Reference" "#PWR06"
 			(at 85.09 102.87 0)
 			(effects
@@
 			)
 		)
-		(property "Value" "GND"
+		(property "Value" "GND_OPA"
 			(at 85.09 101.6 0)
 			(effects
@@
 			(project "headphone_amplifier_v0"
 				(path "/3983550c-3b96-4d77-b5c7-1354f8e757f8/406fb7ac-178d-4932-ad58-7c7a39bfab55"
-					(reference "#PWR08")
-					(unit 1)
-				)
-			)
-		)
-	)
-	(symbol
-		(lib_id "Device:R")
-		(at 124.46 74.93 90)
-		(unit 1)
-		(exclude_from_sim no)
-		(in_bom yes)
-		(on_board yes)
-		(dnp no)
-		(fields_autoplaced yes)
-		(property "Reference" "R8"
-			(at 124.46 68.58 90)
-			(effects
-				(font
-					(size 1.27 1.27)
-				)
-			)
-		)
-		(property "Value" "R"
-			(at 124.46 71.12 90)
-			(effects
-				(font
-					(size 1.27 1.27)
-				)
-			)
-		)
-		(property "Footprint" "Resistor_THT:R_Axial_DIN0309_L9.0mm_D3.2mm_P12.70mm_Horizontal"
-			(at 124.46 76.708 90)
-			(effects
-				(font
-					(size 1.27 1.27)
-				)
-				(hide yes)
-			)
-		)
-		(property "Datasheet" "~"
-			(at 124.46 74.93 0)
-			(effects
-				(font
-					(size 1.27 1.27)
-				)
-				(hide yes)
-			)
-		)
-		(property "Description" "Resistor"
-			(at 124.46 74.93 0)
-			(effects
-				(font
-					(size 1.27 1.27)
-				)
-				(hide yes)
-			)
-		)
-		(pin "1"
-		)
-		(pin "2"
-		)
-		(instances
-			(project "headphone_amplifier_v0"
-				(path "/3983550c-3b96-4d77-b5c7-1354f8e757f8/406fb7ac-178d-4932-ad58-7c7a39bfab55"
-					(reference "R8")
-					(unit 1)
-				)
-			)
-		)
-	)
-	(symbol
-		(lib_id "Device:C")
-		(at 73.66 72.39 90)
-		(unit 1)
-		(exclude_from_sim no)
-		(in_bom yes)
-		(on_board yes)
-		(dnp no)
-		(fields_autoplaced yes)
-		(property "Reference" "C10"
-			(at 73.66 64.77 90)
-			(effects
-				(font
-					(size 1.27 1.27)
-				)
-			)
-		)
-		(property "Value" "0.1u"
-			(at 73.66 67.31 90)
-			(effects
-				(font
-					(size 1.27 1.27)
-				)
-			)
-		)
-		(property "Footprint" ""
-			(at 77.47 71.4248 0)
-			(effects
-				(font
-					(size 1.27 1.27)
-				)
-				(hide yes)
-			)
-		)
-		(property "Datasheet" "~"
-			(at 73.66 72.39 0)
-			(effects
-				(font
-					(size 1.27 1.27)
-				)
-				(hide yes)
-			)
-		)
-		(property "Description" "Unpolarized capacitor"
-			(at 73.66 72.39 0)
-			(effects
-				(font
-					(size 1.27 1.27)
-				)
-				(hide yes)
-			)
-		)
-		(pin "2"
-		)
-		(pin "1"
-		)
-		(instances
-			(project "headphone_amplifier_v0"
-				(path "/3983550c-3b96-4d77-b5c7-1354f8e757f8/406fb7ac-178d-4932-ad58-7c7a39bfab55"
-					(reference "C10")
+					(reference "#PWR06")
 					(unit 1)
 				)
@@
 		(lib_id "Amplifier_Operational:NE5532")
 		(at 109.22 74.93 0)
-		(unit 1)
+		(unit 2)
 		(exclude_from_sim no)
 		(in_bom yes)
@@
 				(path "/3983550c-3b96-4d77-b5c7-1354f8e757f8/406fb7ac-178d-4932-ad58-7c7a39bfab55"
 					(reference "U3")
-					(unit 1)
-				)
-			)
+					(unit 2)
+				)
+			)
