File: power.kicad_sch (KiCad schematic)
At the start: 16 parts, among them J1 Conn_01x03, U1 LM7812_TO220, U2 LM7912_TO220, U3 NE5532

Commit message: complete layout
Parts:
- removed TP1: TP_+12V, TestPoint:TestPoint_THTPad_D1.5mm_Drill0.7mm, symbol Connector:TestPoint
- removed TP2: TP_GND, TestPoint:TestPoint_THTPad_D1.5mm_Drill0.7mm, symbol Connector:TestPoint
- removed TP3: TP_-12V, TestPoint:TestPoint_THTPad_D1.5mm_Drill0.7mm, symbol Connector:TestPoint
- added C10, C9: 0.1u, Capacitor_THT:C_Disc_D5.0mm_W2.5mm_P5.00mm, symbol Device:C
- added C11, C12: 1u, Capacitor_THT:C_Disc_D5.0mm_W2.5mm_P5.00mm, symbol Device:C
- added J6, J7: Conn_01x03, Connector_PinHeader_2.54mm:PinHeader_1x03_P2.54mm_Vertical, symbol Connector_Generic:Conn_01x03
- C1, C2: footprint (none) -> Capacitor_THT:CP_Radial_D12.5mm_P5.00mm
- C3, C4, C7, C8: footprint (none) -> Capacitor_THT:C_Disc_D5.0mm_W2.5mm_P5.00mm
- C5, C6: footprint (none) -> Capacitor_THT:CP_Radial_D5.0mm_P2.50mm
- U1: value LM7812_TO220 -> LM7812
- U2: value LM7912_TO220 -> LM7912
Connections:
- net +12V: now also J6.1 (Pin_1); no longer U3.8 (V+)
- net -12V: now also J6.3 (Pin_3); no longer U3.4 (V-)
- net GND: now also J6.2 (Pin_2)
- net at D1.2: now also J1.1 (Pin_1); no longer J1.3 (Pin_3)
- net VAC: no longer names the net of C2.2, C4.1, D1.4 (-), U2.2 (VI)
- net VAC: no longer D1.3, J1.1 (Pin_1)
- new net: D1.3, J1.3 (Pin_3)
- new net +12V_OPA: C11.2, C9.2, J7.1 (Pin_1), U3.8 (V+)
- new net -12V_OPA: C10.1, C12.1, J7.3 (Pin_3), U3.4 (V-)
- new net GND_OPA: C10.2, C11.1, C12.2, C9.1, J7.2 (Pin_2)
Other:
- moved on the sheet: C1, C2, C3, C4, C5, C6, C7, C8, D1, J1, U1, U2
