File: headphone_amplifier_v0.kicad_pcb (KiCad board)
At the start: 2 copper layers, 75 x 85 mm, 38 parts, among them J1 Conn_01x03, J2 AudioJack3_SwitchTR, J3 Conn_01x03, J4 AudioJack3_SwitchTR, J5 Conn_01x03, J6 Conn_01x03, J7 Conn_01x03, U1 LM7812, U2 LM7912, U3 NE5532

Commit message: revise layout change footprint of RK097 dual
Parts:
- moved REF** 3.00 mm to (169.9, 62.0)
- moved J2 0.14 mm to (119.0, 133.1)
- moved J4 0.12 mm to (150.5, 51.9)
- moved RV1 0.08 mm to (121.5, 55.1)
- moved REF** 0.07 mm to (169.9, 129.9)
Routing:
- net Net-(U3A-+): track 32.2 -> 33.4 mm
- net RIGHT_OUT: track 45.2 -> 46.3 mm
- net GND_OPA: track 261.3 -> 262.2 mm
Other:
- board size 75 x 85 mm -> 74.9 x 84.9 mm
- board text added: "Headphone Amplifier V0"
